File: Documentacion/Plaquetas/Placa V2/PlacaEstimuladorTermico.sch (KiCad schematic (older format))
At the start: 44 parts, among them J2 BorneraGrupoTermistores, J3 BorneraTermistor, J4 BORNERA_VCC, Q1 IRF4905, Q2 IRFZ44N, Q3 IRF4905, Q4 IRFZ44N, Q5 BC337, Q6 BC337, U1 LM2902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

Commit message: Agrego la resistencia en los mos
Parts:
- added R14, R15: R, symbol Device:R
Connections:
- wire segments 157 -> 160
Changed lines of the file:
@@
 Text GLabel 3450 700  1    50   Input ~ 0
 VCC
-Text GLabel 2900 1250 0    50   Input ~ 0
+Text GLabel 2550 1250 0    50   Input ~ 0
 PMOS_FRIO
-Wire Wire Line
-	2900 1250 3150 1250
 $Comp
 L Transistor_BJT:BC337 Q6
@@
 Text GLabel 8100 700  1    50   Input ~ 0
 VCC
-Text GLabel 8400 1250 2    50   Input ~ 0
+Text GLabel 8850 1250 2    50   Input ~ 0
 PMOS_CALOR
 Text GLabel 950  950  0    50   Input ~ 0
@@
 Wire Wire Line
 	3400 5550 3050 5550
+$Comp
+L Device:R R14
+U 1 1 5DA61BA5
+P 2900 1250
+F 0 "R14" V 2693 1250 50  0000 C CNN
+F 1 "R" V 2784 1250 50  0000 C CNN
+F 2 "" V 2830 1250 50  0001 C CNN
+F 3 "~" H 2900 1250 50  0001 C CNN
+	1    2900 1250
+	0    1    1    0
+$EndComp
+Wire Wire Line
+	2750 1250 2550 1250
+Wire Wire Line
+	3050 1250 3150 1250
+$Comp
+L Device:R R15
+U 1 1 5DA8E2C9
+P 8600 1250
+F 0 "R15" V 8393 1250 50  0000 C CNN
+F 1 "R" V 8484 1250 50  0000 C CNN
+F 2 "" V 8530 1250 50  0001 C CNN
+F 3 "~" H 8600 1250 50  0001 C CNN
+	1    8600 1250
+	0    1    1    0
+$EndComp
+Wire Wire Line
+	8450 1250 8400 1250
+Wire Wire Line
+	8750 1250 8850 1250
 $EndSCHEMATC

Commit message: I selected the commercial components values and added to the schematic, I dont know if all the lines are connected correctly so please someone revise
Parts:
- removed unit 2 of U1
- added C12: 100n, symbol Device:C
- added C13, C14: 4.7n, symbol Device:C
- R10: value R -> 82k
- R3, R4, R8: value R -> 39k
- R5: value R -> 27k
- R6: value R -> 3.3k
- R7: value R -> 1k
- R9: value R -> 10k
Connections:
- wire segments 160 -> 187
Other:
- moved on the sheet: A1, C5, C9, J2, R3, R4, R5, U1A

Commit message: Add files via upload
Actualizacion de esquematico: agregada proteccion de bateria
Parts:
- removed C12: 100n, symbol Device:C
- removed C13, C14: 4.7n, symbol Device:C
- added D?: D_Zener, symbol Device:D_Zener
- added D?: DIODE, symbol pspice:DIODE
- added K?: FINDER-34.51, Relay_THT:Relay_SPDT_Finder_34.51_Vertical, symbol Relay:FINDER-34.51
- added R? (x2): R, symbol Device:R
- added RV?: R_POT, symbol Device:R_POT
- added SW?: SW_DIP_x01, symbol Switch:SW_DIP_x01
- added unit 2 of U1
- Q2, Q4: symbol Transistor_FET:IRFZ44N -> PlacaEstimuladorTermico-rescue:IRFZ44N-Transistor_FET
- R10: value 82k -> R
- R3, R4, R8: value 39k -> R
- R5: value 27k -> R
- R6: value 3.3k -> R
- R7: value 1k -> R
- R9: value 10k -> R
- U2, U3: symbol power:MCP1407 -> PlacaEstimuladorTermico-rescue:MCP1407-power
Connections:
- net labels added: inPowerSupply
- wire segments 187 -> 173
- no-connect marks 0 -> 1
Other:
- note added: "Proteccion de la bateria"
- note added: "la red inPowerSupply es el conector que va directo a la fuente de alimentacion.\nEl rele posiblemente convenga comprar un modulo de arduino, que trae el optoacoplador integrado,\nporque es posible que el opamp no pueda entregar corriente como para encender el rele\nEl interruptor seria un pulsador de encendido. Cuando se lo presiona, se enciende el rele y el \nopamp lo mantiene activado despues q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"
- moved on the sheet: A1, C5, C9, J2, R3, R4, R5, U1A

Commit message: Adding indicator lights and values to components
Parts:
- added C10: 4.7n, symbol Device:C
- added D7, D8, D9: LED, symbol Device:LED
- added Q7, Q8, Q9: BC548, Package_TO_SOT_THT:TO-92_Inline, symbol Transistor_BJT:BC548
- added R18, R19, R20: 220, symbol Device:R
- Q2, Q4: symbol PlacaEstimuladorTermico-rescue:IRFZ44N-Transistor_FET -> irfz44n:IRFZ44N
- R10: value R -> 82k
- R14, R15: value R -> 4k7; footprint (none) -> Resistor_SMD:R_0805_2012Metric
- R3, R4, R8: value R -> 39k
- R5: value R -> 27k
- R6: value R -> 3.3k
- R7: value R -> 1k
- R9: value R -> 10k
- U1: footprint (none) -> Package_DIP:DIP-14_W7.62mm_LongPads
- U2, U3: symbol PlacaEstimuladorTermico-rescue:MCP1407-power -> mcp1407:MCP1407
- gave numbers to parts that had none: 7
Connections:
- net labels added: PIN-CAUTION-LED-YELLOW, PIN-READY-LED-GREEN, PIN-WARNING-LED-RED
- wire segments 173 -> 197
Other:
- moved on the sheet: J2, R3, R4, R5, U1A

Commit message: I add all the footprints, the position of the high power mosfets is in acordance with a heatsink that I had
Parts:
- C1, C2: footprint (none) -> Capacitor_THT:CP_Radial_D12.5mm_P5.00mm
- C10, C3, C4, C6: footprint (none) -> Capacitor_THT:C_Disc_D9.0mm_W5.0mm_P10.00mm
- C5, C9: footprint (none) -> Capacitor_THT:C_Radial_D8.0mm_H7.0mm_P3.50mm
- C7: footprint (none) -> Capacitor_THT:C_Radial_D18.0mm_H35.5mm_P7.50mm
- C8: footprint (none) -> Capacitor_THT:C_Disc_D12.0mm_W4.4mm_P7.75mm
- D5: footprint (none) -> Diode_THT:D_5W_P10.16mm_Horizontal
- D6: footprint (none) -> Diode_THT:D_DO-201AE_P12.70mm_Horizontal
- D7, D8, D9, J2, J3, J4, PELTIER1, SW1: footprint (none) -> TerminalBlock:TerminalBlock_bornier-2_P5.08mm
- L1, L2: footprint (none) -> Inductor_THT:L_Radial_D10.0mm_P5.00mm_Neosid_SD12k_style3
- R1, R11, R12, R13, R16, R17, R2: footprint (none) -> Resistor_THT:R_Axial_DIN0309_L9.0mm_D3.2mm_P15.24mm_Horizontal
- R10, R18, R19, R20, R3, R4, R5, R6, R7, R8, R9: footprint (none) -> Resistor_SMD:R_1206_3216Metric
- RV1: footprint (none) -> Potentiometer_THT:Potentiometer_ACP_CA14-H2,5_Horizontal
- U2, U3: footprint (none) -> Package_SO:SOIC-8-1EP_3.9x4.9mm_P1.27mm_EP2.41x3.3mm
