File: Documentacion/Plaquetas/Placa V2/PlacaEstimuladorTermico.sch (KiCad schematic (older format))
At the start: 64 parts, among them J2 BorneraGrupoTermistores, J3 BorneraTermistor, J4 BORNERA_VCC, K1 FINDER-34.51, Q1 IRF4905, Q2 IRFZ44N, Q3 IRF4905, Q4 IRFZ44N, Q5 BC337, Q6 BC337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

Commit message: Add battery level to scheme, protection circuit correction & arranging
Parts:
- added J1: Conn_01x02, Pin_Headers:Pin_Header_Angled_1x02_Pitch2.54mm, symbol Connector_Generic:Conn_01x02
- C11: footprint (none) -> Capacitors_THT:C_Disc_D9.0mm_W5.0mm_P10.00mm
Connections:
- wire segments 202 -> 221
- no-connect marks 1 -> 19
Other:
- note added: "Alimentación Op Amps"
- note added: "Alimentación principal"
- note added: "Driver para el peltier"
- note added: "LEDs indicadores"
- note added: "Medidor de batería"
- note added: "Microcontrolador"
- note added: "Referencia para los Op Amps"
- note added: "Sensor de temperatura del peltier"
- note added: "Sensor de temperatura disipador"
- moved on the sheet: A1, C1, C10, C11, C2, C3, C4, C5, C6, C7, C8, C9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

Commit message: add relay module symbol and footprint, modify mcp1407 symbol
plus updates of these on the schematic
Parts:
- removed K1: FINDER-34.51, Relay_THT:Relay_SPDT_Finder_34.51_Vertical, symbol Relay:FINDER-34.51
- added K1: Modulo_Relé, symbol custom_symbols:Modulo_Relé
Connections:
- wire segments 221 -> 222
Changed lines of the file:
@@
 	-1   0    0    -1
 $EndComp
-Wire Wire Line
-	9670 2070 9670 2290
 Text GLabel 11370 3020 2    50   Input ~ 0
 PWM_FRIO
@@
 	6850 7200 6850 11100
 $Comp
-L Relay:FINDER-34.51 K1
-U 1 1 5DBADF90
-P 1950 8650
-F 0 "K1" V 2517 8650 50  0000 C CNN
-F 1 "FINDER-34.51" V 2426 8650 50  0000 C CNN
-F 2 "Relay_THT:Relay_SPDT_Finder_34.51_Vertical" H 3090 8610 50  0001 C CNN
-F 3 "https://gfinder.findernet.com/public/attachments/34/EN/S34USAEN.pdf" H 1950 8650 50  0001 C CNN
-	1    1950 8650
-	0    1    -1   0
-$EndComp
-$Comp
 L Device:R_POT RV1
 U 1 1 5DBB5534
@@
 	4100 9350 3500 9350
 Wire Wire Line
-	2250 8350 3700 8350
-Wire Wire Line
 	4250 8350 4250 9200
 $Comp
@@
 Wire Wire Line
 	3700 8600 3700 8350
-Connection ~ 3700 8350
 Wire Wire Line
 	3700 8350 4250 8350
@@
 Wire Wire Line
 	2250 9250 2250 8850
-$Comp
-L power:GND #PWR0104
-U 1 1 5DBFFF00
-P 1590 8850
-F 0 "#PWR0104" H 1590 8600 50  0001 C CNN
-F 1 "GND" H 1595 8677 50  0000 C CNN
-F 2 "" H 1590 8850 50  0001 C CNN
-F 3 "" H 1590 8850 50  0001 C CNN
-	1    1590 8850
-	1    0    0    -1
-$EndComp
 Text GLabel 4250 8350 1    50   Input ~ 0
 VCC
-NoConn ~ 2250 8550
-Text GLabel 1650 8450 0    50   Input ~ 0
+Text GLabel 1350 8600 0    50   Input ~ 0
 inPowerSupply
 Text Notes 800  7900 0    50   ~ 0
@@
 Wire Wire Line
 	3700 10250 3700 10290
-Wire Wire Line
-	1650 8850 1590 8850
 Wire Wire Line
 	10420 3470 10570 3470
@@
 NoConn ~ 2900 4600
 Wire Wire Line
-	6370 2070 6370 2350
-Wire Wire Line
 	6170 2870 6370 2870
 Connection ~ 6370 2870
@@
 	-1   0    0    1
 $EndComp
-$Comp
-L power:PWR_FLAG #FLG0103
-U 1 1 5DEABF05
-P 6370 2350
-F 0 "#FLG0103" H 6370 2425 50  0001 C CNN
-F 1 "PWR_FLAG" V 6370 2477 50  0000 L CNN
-F 2 "" H 6370 2350 50  0001 C CNN
-F 3 "~" H 6370 2350 50  0001 C CNN
-	1    6370 2350
-	0    -1   -1   0
-$EndComp
-Connection ~ 6370 2350
-Wire Wire Line
-	6370 2350 6370 2870
-$Comp
-L power:PWR_FLAG #FLG0104
-U 1 1 5DEACECF
-P 9670 2290
-F 0 "#FLG0104" H 9670 2365 50  0001 C CNN
-F 1 "PWR_FLAG" V 9670 2418 50  0000 L CNN
-F 2 "" H 9670 2290 50  0001 C CNN
-F 3 "~" H 9670 2290 50  0001 C CNN
-	1    9670 2290
-	0    1    1    0
-$EndComp
-Connection ~ 9670 2290
-Wire Wire Line
-	9670 2290 9670 2970
 Wire Wire Line
 	4490 3610 4830 3610
@@
 	2440 9250 2400 9250
 Connection ~ 2400 9250
+NoConn ~ 1350 8850
+Wire Wire Line
+	2250 8600 2900 8600
+Wire Wire Line
+	2900 8600 2900 8350
+Wire Wire Line
+	2900 8350 3700 8350
+Connection ~ 3700 8350
+$Comp
+L power:GND #PWR017
+U 1 1 5E3E5CAB
+P 2400 8350
+F 0 "#PWR017" H 2400 8100 50  0001 C CNN
+F 1 "GND" V 2405 8222 50  0000 R CNN
+F 2 "" H 2400 8350 50  0001 C CNN
+F 3 "" H 2400 8350 50  0001 C CNN
+	1    2400 8350
+	0    -1   -1   0
+$EndComp
+Wire Wire Line
+	2250 8350 2400 8350
+Text GLabel 1210 8350 0    50   Input ~ 0
+VCC
+Wire Wire Line
+	1350 8350 1210 8350
+$Comp
+L custom_symbols:Modulo_Relé K1
+U 1 1 5E40A870
+P 1800 9050
+F 0 "K1" H 1800 8035 50  0000 C CNN
+F 1 "Modulo_Relé" H 1800 8126 50  0000 C CNN
+F 2 "" H 1800 9050 50  0001 C CNN
+F 3 "" H 1800 9050 50  0001 C CNN
+	1    1800 9050
+	-1   0    0    1
+$EndComp
+Wire Wire Line
+	6370 2070 6370 2870
+Wire Wire Line
+	9670 2070 9670 2970
 $EndSCHEMATC
