File: Documentacion/Plaquetas/Placa V2/_autosave-PlacaEstimuladorTermico.sch (KiCad schematic (older format))
At the start: 64 parts, among them J2 BorneraGrupoTermistores, J3 BorneraTermistor, J4 BORNERA_VCC, K1 FINDER-34.51, Q1 IRF4905, Q2 IRFZ44N, Q3 IRF4905, Q4 IRFZ44N, Q5 BC337, Q6 BC337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

Commit message: I designed the pcb, it was my first try so please check every wire
Parts:
- C10: footprint Capacitor_THT:C_Disc_D9.0mm_W5.0mm_P10.00mm -> Capacitor_THT:C_Disc_D7.0mm_W2.5mm_P5.00mm
- C11: footprint (none) -> Capacitor_THT:C_Disc_D7.0mm_W2.5mm_P5.00mm
Changed lines of the file:
@@
 F 0 "C10" H 7065 5696 50  0000 L CNN
 F 1 "4.7n" H 7065 5605 50  0000 L CNN
-F 2 "Capacitor_THT:C_Disc_D9.0mm_W5.0mm_P10.00mm" H 6988 5500 50  0001 C CNN
+F 2 "Capacitor_THT:C_Disc_D7.0mm_W2.5mm_P5.00mm" H 6988 5500 50  0001 C CNN
 F 3 "~" H 6950 5650 50  0001 C CNN
 	1    6950 5650
@@
 F 0 "C11" H 5265 5246 50  0000 L CNN
 F 1 "4.7n" H 5265 5155 50  0000 L CNN
-F 2 "" H 5188 5050 50  0001 C CNN
+F 2 "Capacitor_THT:C_Disc_D7.0mm_W2.5mm_P5.00mm" H 5188 5050 50  0001 C CNN
 F 3 "~" H 5150 5200 50  0001 C CNN
 	1    5150 5200
