File: Documentacion/Plaquetas/Placa control/PlacaEstimuladorTermico.kicad_pcb (KiCad board)
At the start: 2 copper layers, 172.2 x 74.2 mm, 26 parts, among them J11 Conn_01x03_Male, J12 Conn_01x02_Male, J13 Conn_01x02_Male, J2 DB9_Female_MountingHoles, J3 Screw_Terminal_01x02, J4 Conn_01x06_Male, J7 Conn_02x05_Counter_Clockwise, J9 Conn_01x06_Male, Q7 BC548, Q8 BC548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

Commit message: changes in the schematic and pcb
Parts:
- added C4: 2.2n, Capacitor_SMD:C_1206_3216Metric_Pad1.42x1.75mm_HandSolder, F.Cu at (206.2, 113.3)
- added C6: 2.2n, Capacitor_SMD:C_1206_3216Metric_Pad1.42x1.75mm_HandSolder, F.Cu at (204.2, 97.5)
- added J14: Conn_01x03_Male, Connector_PinHeader_2.54mm:PinHeader_1x03_P2.54mm_Vertical, F.Cu at (128.0, 78.7)
- added R4: 10k, Resistor_SMD:R_1206_3216Metric, F.Cu at (221.0, 105.7)
- added R5: 10k, Resistor_SMD:R_1206_3216Metric, F.Cu at (217.9, 108.7)
- C11: value 47n -> 4.7n
- R3: value 20k -> 10k
- moved J12 15.7 mm to (109.2, 78.7), turned to 90 degrees
- moved J13 6.10 mm to (118.9, 78.7), turned to 90 degrees
Connections:
- net PIN_SENSOR_TEMPERATURA_DISIPADOR renamed PIN_SENSOR_TEMPERATURA_1
- net PIN_SENSOR_TEMPERATURA_SUPERFICIAL renamed PIN_SENSOR_TEMPERATURA_2
- net term_disip_1C renamed term_1_1C
- A1 pad 5: Net-(A1-Pad5) -> SENSOR_PUMP
- A1 pad 6: Net-(A1-Pad6) -> SENSOR_FAN
- J11 pad 1: fan_in_2C -> pump_sensor_C
- J12 pad 1: term_pelt_1C -> term_2_1C
- J12 pad 2: term_pelt_2C -> term_2_2C
- J13 pad 2: term_disip_2C -> term_1_2C
- J2 pad 0: fan_2C -> Net-(J2-Pad0)
- J2 pad 1: term_pelt_1C -> fan_sensor_C
- J2 pad 2: term_pelt_2C -> term_1_2C
- J2 pad 4: term_disip_2C -> term_2_2C
- J2 pad 5: fan_1C -> term_2_1C
- J2 pad 6: fan_in_2C -> fan_1C
- J2 pad 9: fan_1C -> pump_sensor_C
- J7 pad 3: fan_in_2 -> SENSOR_PUMP
- J7 pad 8: VCC -> SENSOR_FAN
Routing:
- net fan_in_2: track 59.6 -> 0.00 mm, vias 3 -> 0
- net SENSOR_FAN: track 0.00 -> 56.2 mm, vias 0 -> 2
- net fan_in_2C: track 53.1 -> 0.00 mm
- net SENSOR_PUMP: track 0.00 -> 43.6 mm, vias 0 -> 3
- net fan_1C: track 19.9 -> 55.9 mm
- net fan_2C: track 54.0 -> 78.9 mm
- net pump_sensor_C: track 0.00 -> 19.5 mm
- net fan_sensor_C: track 0.00 -> 16.3 mm
- net term_pelt_2C: track 15.1 -> 0.00 mm
- net term_pelt_1C: track 15.0 -> 0.00 mm
- net term_1_2C: track 0.00 -> 14.7 mm
- net term_2_1C: track 0.00 -> 13.1 mm
- net term_disip_2C: track 13.0 -> 0.00 mm
- net term_2_2C: track 0.00 -> 13.0 mm
- net fan_2: track 303.4 -> 311.5 mm
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Other:
- outline, holes or cut-outs redrawn
- board text added: "Cooler FAN"
- board text added: "Cooler PUMP"
- board text removed: "Cooler"
