File: Documentacion/Plaquetas/Placa control/PlacaEstimuladorTermico3.sch (KiCad schematic (older format))
At the start: 35 parts, among them J10 Conn_01x06_Female, J11 Conn_01x03_Male, J12 Conn_01x02_Male, J13 Conn_01x02_Male, J14 Conn_01x03_Male, J2 DB9_Female_MountingHoles, J3 Screw_Terminal_01x02, J4 Conn_01x06_Male, J7 Conn_02x05_Counter_Clockwise, J9 Conn_01x06_Male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

Commit message: changes in the schematic and pcb
Parts:
- removed C4, C6: 2.2n, Capacitor_SMD:C_1206_3216Metric_Pad1.42x1.75mm_HandSolder, symbol Device:C
- removed J14: Conn_01x03_Male, Connector_PinHeader_2.54mm:PinHeader_1x03_P2.54mm_Vertical, symbol Connector:Conn_01x03_Male
- removed R4, R5: 10k, symbol Device:R
- C11: value 4.7n -> 47n
- R3: value 10k -> 20k
Connections:
- net labels added: PIN_SENSOR_TEMPERATURA_DISIPADOR, PIN_SENSOR_TEMPERATURA_SUPERFICIAL, fan_in_2C, term_disip_1, term_disip_1C, term_disip_2, term_disip_2C, term_pelt_1, term_pelt_1C, term_pelt_2, term_pelt_2C
- net labels removed: PIN_SENSOR_TEMPERATURA_1, PIN_SENSOR_TEMPERATURA_2, SENSOR_FAN, SENSOR_PUMP, fan_sensor, fan_sensor_C, pump_sensor, pump_sensor_C, term_1_1, term_1_1C, term_1_2, term_1_2C, term_2_1, term_2_1C, term_2_2, term_2_2C
- wire segments 223 -> 209
- no-connect marks 14 -> 16
Other:
- note removed: "Sensores Water Cooling\n"
- moved on the sheet: J12, J13, J2
