File: Documentacion/Plaquetas/Placa control/placa control.sch (KiCad schematic (older format))
At the start: 44 parts, among them J1 Conn_01x02_Male, J10 Conn_01x06_Female, J11 Conn_01x03_Male, J12 Conn_01x03_Male, J13 Conn_01x03_Male, J2 DB9_Female_MountingHoles, J3 Screw_Terminal_01x02, J4 Conn_01x06_Male, J5 Conn_01x02_Male, J6 Conn_01x04_Male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

Commit message: Added capacitor to buzzer transistor's base, changed 7805 diode side
changed connector wire order,
added proof of concept layout for single sided board,
removed outdated and cache files
Parts:
- added C1: 2u, Capacitor_THT:C_Disc_D4.7mm_W2.5mm_P5.00mm, symbol Device:C
- C10, C11, C2, C3, C4, C6, C9: footprint Capacitor_SMD:C_1206_3216Metric_Pad1.42x1.75mm_HandSolder -> Capacitor_THT:C_Disc_D4.7mm_W2.5mm_P5.00mm
- R1, R18, R19, R2, R20, R4, R5, R6, R7: footprint Resistor_SMD:R_1206_3216Metric -> Resistor_THT:R_Axial_DIN0414_L11.9mm_D4.5mm_P15.24mm_Horizontal
Connections:
- wire segments 240 -> 238
- no-connect marks 14 -> 16
Other:
- moved on the sheet: C2, C3, D1, U1

Commit message: Possible route design, swapped display connector pins
Other:
- moved on the sheet: R6, R7
Changed lines of the file:
@@
 	1    0    0    -1
 $EndComp
+Text GLabel 4620 5835 2    50   Input ~ 0
+SDA-DISPLAY
 Text GLabel 4620 5735 2    50   Input ~ 0
-SDA-DISPLAY
-Text GLabel 4620 5835 2    50   Input ~ 0
 SCL-DISPLAY
 Text GLabel 4980 5235 2    50   Input ~ 0
@@
 L Device:R R7
 U 1 1 5EE92728
+P 4300 5490
+F 0 "R7" H 4370 5536 50  0000 L CNN
+F 1 "10k" H 4370 5445 50  0000 L CNN
+F 2 "Resistor_THT:R_Axial_DIN0414_L11.9mm_D4.5mm_P15.24mm_Horizontal" V 4230 5490 50  0001 C CNN
+F 3 "~" H 4300 5490 50  0001 C CNN
+	1    4300 5490
+	1    0    0    -1
+$EndComp
+$Comp
+L Device:R R6
+U 1 1 5EE931B7
 P 4550 5490
-F 0 "R7" H 4620 5536 50  0000 L CNN
+F 0 "R6" H 4620 5536 50  0000 L CNN
 F 1 "10k" H 4620 5445 50  0000 L CNN
 F 2 "Resistor_THT:R_Axial_DIN0414_L11.9mm_D4.5mm_P15.24mm_Horizontal" V 4480 5490 50  0001 C CNN
@@
 	1    0    0    -1
 $EndComp
-$Comp
-L Device:R R6
-U 1 1 5EE931B7
-P 4300 5490
-F 0 "R6" H 4370 5536 50  0000 L CNN
-F 1 "10k" H 4370 5445 50  0000 L CNN
-F 2 "Resistor_THT:R_Axial_DIN0414_L11.9mm_D4.5mm_P15.24mm_Horizontal" V 4230 5490 50  0001 C CNN
-F 3 "~" H 4300 5490 50  0001 C CNN
-	1    4300 5490
-	1    0    0    -1
-$EndComp

Commit message: Changed pump and fan sensor pins, routed accordingly, shrunk board size
Connections:
- wire segments 238 -> 236
Changed lines of the file:
@@
 	1    0    0    -1
 $EndComp
-Text GLabel 5400 2430 2    50   Input ~ 0
-PIN_SENSOR_TEMPERATURA_2
-Wire Wire Line
-	5100 2330 5400 2330
 $Comp
 L Device:R R3
@@
 Wire Wire Line
 	6275 4320 6525 4320
-Text GLabel 5400 2330 2    50   Input ~ 0
-PIN_SENSOR_TEMPERATURA_1
 Text GLabel 770  880  0    50   Input ~ 0
 VCC
@@
 	1840 3535 1905 3535
 Connection ~ 1445 4040
-$Comp
-L custom_symbols:Arduino_Nano_v2.x A1
-U 1 1 5DB11DC8
-P 4600 1730
-F 0 "A1" H 4600 641 50  0000 C CNN
-F 1 "Arduino_Nano_v3.x" H 4600 550 50  0000 C CNN
-F 2 "Module:Arduino_Nano" H 4750 780 50  0001 L CNN
-F 3 "http://www.mouser.com/pdfdocs/Gravitech_Arduino_Nano3_0.pdf" H 4600 730 50  0001 C CNN
-	1    4600 1730
-	1    0    0    -1
-$EndComp
 Text GLabel 800  3535 0    50   Input ~ 0
 REF_5
@@
 Wire Wire Line
 	4600 3665 4760 3665
-Wire Wire Line
-	4100 1335 4100 1330
-Wire Wire Line
-	3965 1520 3965 1430
-Wire Wire Line
-	3965 1430 4100 1430
-Text GLabel 3740 1335 0    50   Input ~ 0
-SENSOR_PUMP
-Text GLabel 3965 1520 0    50   Input ~ 0
-SENSOR_FAN
-Wire Wire Line
-	3740 1335 4100 1335
 Wire Wire Line
 	4355 3665 4355 3745
@@
 $EndComp
 Wire Wire Line
-	5100 2430 5400 2430
-Wire Wire Line
 	5100 1930 5400 1930
 Wire Wire Line
@@
 Text GLabel 4045 1830 0    50   Input ~ 0
 PIN-HOT-LED-YELLOW
-NoConn ~ 5100 1730
-NoConn ~ 5100 1830
 Wire Wire Line
 	3595 2130 4100 2130
@@
 Wire Wire Line
 	10095 3860 10130 3860
+Wire Wire Line
+	5460 1830 5100 1830
+Text GLabel 5235 1730 2    50   Input ~ 0
+SENSOR_PUMP
+Wire Wire Line
+	5235 1730 5100 1730
+Wire Wire Line
+	5100 2430 5400 2430
+Text GLabel 5400 2330 2    50   Input ~ 0
+PIN_SENSOR_TEMPERATURA_1
+Wire Wire Line
+	5100 2330 5400 2330
+Text GLabel 5400 2430 2    50   Input ~ 0
+PIN_SENSOR_TEMPERATURA_2
+Text GLabel 5460 1830 2    50   Input ~ 0
+SENSOR_FAN
+NoConn ~ 4100 1430
+$Comp
+L custom_symbols:Arduino_Nano_v2.x A1
+U 1 1 5DB11DC8
+P 4600 1730
+F 0 "A1" H 4600 641 50  0000 C CNN
+F 1 "Arduino_Nano_v3.x" H 4600 550 50  0000 C CNN
+F 2 "Module:Arduino_Nano" H 4750 780 50  0001 L CNN
+F 3 "http://www.mouser.com/pdfdocs/Gravitech_Arduino_Nano3_0.pdf" H 4600 730 50  0001 C CNN
+	1    4600 1730
+	1    0    0    -1
+$EndComp
+NoConn ~ 4100 1330
 $EndSCHEMATC

Commit message: Possible design, swapped sda and scl connector pins
Parts:
- A1: footprint Module:Arduino_Nano -> custom_footprints:Arduino_Nano
- J1, J5, J8: footprint Connector_PinHeader_2.54mm:PinHeader_1x02_P2.54mm_Vertical -> custom_footprints:PinHeader_1x02_P2.54mm_Vertical
- J6: footprint Connector_PinHeader_2.54mm:PinHeader_1x04_P2.54mm_Vertical -> custom_footprints:PinHeader_1x04_P2.54mm_Vertical
- J9: footprint Connector_PinHeader_2.54mm:PinHeader_1x08_P2.54mm_Vertical -> custom_footprints:PinHeader_1x08_P2.54mm_Vertical
Changed lines of the file:
@@
 F 0 "J1" H 2303 6976 50  0000 C CNN
 F 1 "Conn_01x02_Male" H 2303 6885 50  0000 C CNN
-F 2 "Connector_PinHeader_2.54mm:PinHeader_1x02_P2.54mm_Vertical" H 2195 6795 50  0001 C CNN
+F 2 "custom_footprints:PinHeader_1x02_P2.54mm_Vertical" H 2195 6795 50  0001 C CNN
 F 3 "~" H 2195 6795 50  0001 C CNN
 	1    2195 6795
@@
 F 0 "J5" H 10265 3400 50  0000 C CNN
 F 1 "Conn_01x02_Male" H 10265 3500 50  0000 C CNN
-F 2 "Connector_PinHeader_2.54mm:PinHeader_1x02_P2.54mm_Vertical" H 10630 3555 50  0001 C CNN
+F 2 "custom_footprints:PinHeader_1x02_P2.54mm_Vertical" H 10630 3555 50  0001 C CNN
 F 3 "~" H 10630 3555 50  0001 C CNN
 	1    10630 3555
@@
 F 0 "J9" V 8920 708 50  0000 C CNN
 F 1 "Conn_01x08_Male" V 9011 708 50  0000 C CNN
-F 2 "Connector_PinHeader_2.54mm:PinHeader_1x08_P2.54mm_Vertical" H 9085 780 50  0001 C CNN
+F 2 "custom_footprints:PinHeader_1x08_P2.54mm_Vertical" H 9085 780 50  0001 C CNN
 F 3 "~" H 9085 780 50  0001 C CNN
 	1    9085 780
@@
 F 0 "J6" H 3758 6016 50  0000 C CNN
 F 1 "Conn_01x04_Male" H 3758 5925 50  0000 C CNN
-F 2 "Connector_PinHeader_2.54mm:PinHeader_1x04_P2.54mm_Vertical" H 3650 5735 50  0001 C CNN
+F 2 "custom_footprints:PinHeader_1x04_P2.54mm_Vertical" H 3650 5735 50  0001 C CNN
 F 3 "~" H 3650 5735 50  0001 C CNN
 	1    3650 5735
 	1    0    0    -1
 $EndComp
+Text GLabel 4620 5735 2    50   Input ~ 0
+SDA-DISPLAY
 Text GLabel 4620 5835 2    50   Input ~ 0
-SDA-DISPLAY
-Text GLabel 4620 5735 2    50   Input ~ 0
 SCL-DISPLAY
 Text GLabel 4980 5235 2    50   Input ~ 0
@@
 	8470 3745 8255 3745
 NoConn ~ 2165 5020
-Text GLabel 2265 5320 2    50   Input ~ 0
+Text GLabel 1520 5395 0    50   Input ~ 0
 VCC
 Wire Wire Line
@@
 L power:GND #PWR0109
 U 1 1 5EC8211E
-P 1520 5395
-F 0 "#PWR0109" H 1520 5145 50  0001 C CNN
-F 1 "GND" H 1525 5222 50  0000 C CNN
-F 2 "" H 1520 5395 50  0001 C CNN
-F 3 "" H 1520 5395 50  0001 C CNN
-	1    1520 5395
+P 2265 5320
+F 0 "#PWR0109" H 2265 5070 50  0001 C CNN
+F 1 "GND" H 2270 5147 50  0000 C CNN
+F 2 "" H 2265 5320 50  0001 C CNN
+F 3 "" H 2265 5320 50  0001 C CNN
+	1    2265 5320
 	1    0    0    -1
 $EndComp
@@
 F 0 "J8" V 2315 5330 50  0000 C CNN
 F 1 "Conn_01x02_Male" V 2395 5335 50  0000 C CNN
-F 2 "Connector_PinHeader_2.54mm:PinHeader_1x02_P2.54mm_Vertical" H 1970 5380 50  0001 C CNN
+F 2 "custom_footprints:PinHeader_1x02_P2.54mm_Vertical" H 1970 5380 50  0001 C CNN
 F 3 "~" H 1970 5380 50  0001 C CNN
 	1    1970 5380
@@
 F 0 "A1" H 4600 641 50  0000 C CNN
 F 1 "Arduino_Nano_v3.x" H 4600 550 50  0000 C CNN
-F 2 "Module:Arduino_Nano" H 4750 780 50  0001 L CNN
+F 2 "custom_footprints:Arduino_Nano" H 4750 780 50  0001 L CNN
 F 3 "http://www.mouser.com/pdfdocs/Gravitech_Arduino_Nano3_0.pdf" H 4600 730 50  0001 C CNN
 	1    4600 1730
