File: Documentacion/Plaquetas/Placa control/placa control.kicad_pcb (KiCad board)
At the start: 2 copper layers, 93.8 x 94.5 mm, 44 parts, among them J1 Conn_01x02_Male, J10 Conn_01x06_Female, J11 Conn_01x03_Male, J12 Conn_01x03_Male, J13 Conn_01x03_Male, J2 DB9_Female_MountingHoles, J3 Screw_Terminal_01x02, J4 Conn_01x06_Male, J5 Conn_01x02_Male, J6 Conn_01x04_Male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

Commit message: changed buzzer to common collector mode
Parts:
- moved J1 9.12 mm to (43.4, 158.0)
- moved J13 6.86 mm to (50.2, 157.9)
- moved Q1 4.68 mm to (66.7, 80.0), turned to 90 degrees
- moved J5 0.28 mm to (58.4, 65.3)
Connections:
- J5 pad 1: Net-(J5-Pad1) -> GND
- J5 pad 2: REF_5 -> Net-(J5-Pad2)
- Q1 pad 1: Net-(J5-Pad1) -> REF_5
- Q1 pad 3: GND -> Net-(J5-Pad2)
Routing:
- net REF_5: track 124.0 -> 142.1 mm
- net pump_sensor_C: track 45.4 -> 29.0 mm
- net Net-(J5-Pad1): track 16.4 -> 0.00 mm
- net Net-(J5-Pad2): track 0.00 -> 14.5 mm
- net Net-(A1-Pad17): track 0.00 -> 6.03 mm
- net Net-(A1-Pad16): track 0.00 -> 6.03 mm
- net Net-(A1-Pad7): track 0.00 -> 5.78 mm
- net Net-(A1-Pad6): track 0.00 -> 5.78 mm
- net Net-(A1-Pad5): track 0.00 -> 5.78 mm
- net Net-(A1-Pad2): track 0.00 -> 5.78 mm
- net Net-(A1-Pad15): track 0.00 -> 5.78 mm
- net Net-(A1-Pad1): track 0.00 -> 5.78 mm
- net Net-(A1-Pad3): track 0.00 -> 5.64 mm
- net VCC_C: track 39.1 -> 43.4 mm
- net GND: track 395.3 -> 391.1 mm
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Other:
- board size 93.8 x 94.5 mm -> 114.3 x 143.3 mm
